File: CE/advanced-BLE-CELL/advanced-BLE-CELL.kicad_pcb (KiCad board)
At the start: 4 copper layers, 65 x 56 mm, 24 parts, among them J3 40HAT, J6 CONN_02X02, J9 CONN_01X02, Q1 DMG2305UX, Q2 DMMT5401, U1 nRF52840, U2 CAT24C32, U3 BG96

Commit message: asdf
Parts:
- H5, H6, H7, H8: footprint ABC:4881 -> ABC:4881-Top; moved to B.Cu

Commit message: Asd
Parts:
- U1: moved to B.Cu
- moved U1 0.41 mm to (111.7, 83.2)
