File: CE/advanced-BLE-CELL/advanced-BLE-CELL.kicad_pcb (KiCad board)
At the start: 4 copper layers, 65 x 56 mm, 24 parts, among them J3 40HAT, J6 CONN_02X02, J9 CONN_01X02, Q1 DMG2305UX, Q2 DMMT5401, U1 nRF52840, U2 CAT24C32, U3 BG96

Commit message: ASFd
Parts:
- J3: footprint Connector_PinSocket_2.54mm:PinSocket_2x20_P2.54mm_Vertical -> ABC:PinSocket_2x20_P2.54mm_Vertical-CENTER
- moved J3 23.7 mm to (110.5, 63.8)
- moved U3 1.40 mm to (111.0, 100.2)
- moved H2 0.99 mm to (139.5, 63.5)
- moved H1 0.97 mm to (81.5, 63.5)
- moved H3 0.63 mm to (81.5, 113.0)
- moved H4 0.61 mm to (139.5, 113.0)
Routing:
- net /ID_SC_EEPROM: track 11.7 -> 9.76 mm
Other:
- board size 65 x 56 mm -> 65 x 56.5 mm

Commit message: asf
Parts:
- added N1: Rasp Pi 3d Model, ABC:KiCad-Logo_5mm_SilkScreen-rpi-module, B.Cu at (134.5, 71.0)
- U1: moved to F.Cu
- moved H7 10.2 mm to (116.2, 80.0)
- moved H8 8.51 mm to (117.5, 112.5)
- moved U3 4.81 mm to (108.2, 96.2)
- moved U1 4.73 mm to (108.8, 79.5)
- moved H5 4.60 mm to (101.2, 79.8)
- moved H6 2.30 mm to (100.2, 112.5)
- moved J3 0.25 mm to (110.8, 63.8)
Other:
- outline, holes or cut-outs redrawn

Commit message: das
Parts:
- added J1: Conn_01x02_Male, Connector_JST:JST_PH_S2B-PH-SM4-TB_1x02-1MP_P2.00mm_Horizontal, F.Cu at (102.4, 78.6)
- added P1: USB_C_Plug_USB2.0, Connector_USB:USB_C_Receptacle_Palconn_UTC16-G, F.Cu at (117.4, 102.0)
- moved J6 21.6 mm to (72.5, 71.2)
- moved Q1 21.6 mm to (66.1, 67.1)
- moved Q2 21.6 mm to (66.5, 70.6)
- moved R23 21.6 mm to (65.4, 74.1)
- moved R24 21.6 mm to (67.7, 74.1)
- moved R7 21.6 mm to (71.2, 74.0)
- moved R9 21.6 mm to (71.1, 65.9)
- moved R11 16.0 mm to (136.1, 74.5)
- moved R29 16.0 mm to (130.4, 71.9)
- moved R6 16.0 mm to (130.4, 68.6)
- moved R8 16.0 mm to (130.4, 70.2)
- moved U2 16.0 mm to (136.1, 70.6)
- moved J9 16.0 mm to (129.7, 74.6)
- moved U1 12.3 mm to (117.4, 88.2)
- moved H5 6.97 mm to (94.5, 78.0)
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Other:
- outline, holes or cut-outs redrawn
