File: CE/advanced-BLE-CELL/advanced-BLE-CELL.sch (KiCad schematic (older format))
At the start: 25 parts, among them J3 40HAT, J6 CONN_02X02, J9 CONN_01X02, Q1 DMG2305UX, Q2 DMMT5401, U1 nRF52840, U2 CAT24C32, U3 BG96

Commit message: ASFd
Parts:
- H5, H6, H7, H8: footprint ABC:4881 -> ABC:4881-Top
- J3: footprint Connector_PinSocket_2.54mm:PinSocket_2x20_P2.54mm_Vertical -> ABC:PinSocket_2x20_P2.54mm_Vertical-CENTER
Other:
- moved on the sheet: N1
Changed lines of the file:
@@
 F 0 "J3" H 2950 2350 50  0000 C CNN
 F 1 "40HAT" H 2300 2350 50  0000 C CNN
-F 2 "Connector_PinSocket_2.54mm:PinSocket_2x20_P2.54mm_Vertical" H 2600 2450 50  0001 C CNN
+F 2 "ABC:PinSocket_2x20_P2.54mm_Vertical-CENTER" H 2600 2450 50  0001 C CNN
 F 3 "" H 1900 2250 50  0000 C CNN
 	1    2600 2250
@@
 L Mechanical:Housing N1
 U 1 1 5FDFAE6F
-P 15650 1700
-F 0 "N1" H 15803 1734 50  0000 L CNN
-F 1 "Rasp Pi 3d Model" H 15803 1643 50  0000 L CNN
-F 2 "" H 15700 1750 50  0001 C CNN
-F 3 "~" H 15700 1750 50  0001 C CNN
-	1    15650 1700
+P 15700 2000
+F 0 "N1" H 15853 2034 50  0000 L CNN
+F 1 "Rasp Pi 3d Model" H 15853 1943 50  0000 L CNN
+F 2 "" H 15750 2050 50  0001 C CNN
+F 3 "~" H 15750 2050 50  0001 C CNN
+	1    15700 2000
 	1    0    0    -1
 $EndComp
@@
 F 0 "H5" H 9250 6550 60  0000 C CNN
 F 1 "4881 SMT Mounts" H 9400 6300 60  0000 C CNN
-F 2 "ABC:4881" H 9300 6450 60  0001 C CNN
+F 2 "ABC:4881-Top" H 9300 6450 60  0001 C CNN
 F 3 "" H 9300 6450 60  0001 C CNN
 	1    9400 6450
@@
 F 0 "H7" H 10350 6550 60  0000 C CNN
 F 1 "4881 SMT Mounts" H 10500 6300 60  0000 C CNN
-F 2 "ABC:4881" H 10400 6450 60  0001 C CNN
+F 2 "ABC:4881-Top" H 10400 6450 60  0001 C CNN
 F 3 "" H 10400 6450 60  0001 C CNN
 	1    10500 6450
@@
 F 0 "H6" H 9250 7050 60  0000 C CNN
 F 1 "4881 SMT Mounts" H 9400 6800 60  0000 C CNN
-F 2 "ABC:4881" H 9300 6950 60  0001 C CNN
+F 2 "ABC:4881-Top" H 9300 6950 60  0001 C CNN
 F 3 "" H 9300 6950 60  0001 C CNN
 	1    9400 6950
@@
 F 0 "H8" H 10350 7050 60  0000 C CNN
 F 1 "4881 SMT Mounts" H 10500 6800 60  0000 C CNN
-F 2 "ABC:4881" H 10400 6950 60  0001 C CNN
+F 2 "ABC:4881-Top" H 10400 6950 60  0001 C CNN
 F 3 "" H 10400 6950 60  0001 C CNN
 	1    10500 6950

Commit message: asf
Parts:
- N1: footprint (none) -> ABC:KiCad-Logo_5mm_SilkScreen-rpi-module
Changed lines of the file:
@@
 F 0 "N1" H 15853 2034 50  0000 L CNN
 F 1 "Rasp Pi 3d Model" H 15853 1943 50  0000 L CNN
-F 2 "" H 15750 2050 50  0001 C CNN
+F 2 "ABC:KiCad-Logo_5mm_SilkScreen-rpi-module" H 15750 2050 50  0001 C CNN
 F 3 "~" H 15750 2050 50  0001 C CNN
 	1    15700 2000

Commit message: das
Parts:
- added J1: Conn_01x02_Male, Connector_JST:JST_PH_S2B-PH-SM4-TB_1x02-1MP_P2.00mm_Horizontal, symbol Connector:Conn_01x02_Male
- added P1: USB_C_Plug_USB2.0, Connector_USB:USB_C_Receptacle_Palconn_UTC16-G, symbol Connector:USB_C_Plug_USB2.0
Connections:
- new net: P1.A1 (GND), P1.A12 (GND), P1.B1 (GND), P1.B12 (GND)
- new net: P1.A4 (VBUS), P1.A9 (VBUS), P1.B4 (VBUS), P1.B9 (VBUS)
Changed lines of the file:
@@
+	1    0    0    -1
+$EndComp
+$Comp
+L Connector:USB_C_Plug_USB2.0 P1
+U 1 1 5FF3FC99
+P 17700 8100
+F 0 "P1" H 17807 8967 50  0000 C CNN
+F 1 "USB_C_Plug_USB2.0" H 17807 8876 50  0000 C CNN
+F 2 "Connector_USB:USB_C_Receptacle_Palconn_UTC16-G" H 17850 8100 50  0001 C CNN
+F 3 "https://www.usb.org/sites/default/files/documents/usb_type-c.zip" H 17850 8100 50  0001 C CNN
+	1    17700 8100
+	1    0    0    -1
+$EndComp
+$Comp
+L Connector:Conn_01x02_Male J1
+U 1 1 5FF4F6D5
+P 18300 9250
+F 0 "J1" H 18408 9431 50  0000 C CNN
+F 1 "Conn_01x02_Male" H 18408 9340 50  0000 C CNN
+F 2 "Connector_JST:JST_PH_S2B-PH-SM4-TB_1x02-1MP_P2.00mm_Horizontal" H 18300 9250 50  0001 C CNN
+F 3 "~" H 18300 9250 50  0001 C CNN
+	1    18300 9250
 	1    0    0    -1
 $EndComp
